File: MicroFLiC_DAC_1_0.kicad_pcb (KiCad board)
At the start: 4 copper layers, 49.8 x 49.8 mm, 122 parts, among them P1 CONN_02X04, P2 CONN_02X04, P3 SMA, P4 SMA, P5 SMA, P6 SMA, P7 CONN_01X02, P8 CONN_01X02, U1 DAC8734, U10 TPS7A4901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

Commit message: Final production board v1.0
Parts:
- added A1: JMP, jakub:JMP, F.Cu at (134.4, 124.5)
- C16, C17, C22, C23, C27, C29, C33, C35: value 100p -> 470p
- P1: value CONN_02X04 -> 2x4_MicroMaTch
- P2: value CONN_02X04 -> 2x4_HEADER
- P7: value CONN_01X02 -> 1x2_HEADER
- P8: value CONN_01X02 -> 1x2_SOCKET
- R23, R24: value 49R9 -> 49R9/0.1%/125mW
- R6, R7, R8, R9: value 1k -> 1k/0.05%/125mW
Connections:
- C11 pad 2: GNDA -> GND
- C12 pad 2: GNDA -> GND
- C67 pad 2: GNDA -> GND
- P2 pad 2: GNDA -> GND
- R1 pad 2: GNDA -> GND
- R2 pad 2: GNDA -> GND
- R3 pad 2: GNDA -> GND
- R4 pad 2: GNDA -> GND
- U1 pad 11: GNDA -> GND
- U15 pad 9: GNDA -> GND
Routing:
- net GNDA: track 1110.5 -> 979.9 mm, vias 20 -> 15
- net GND: track 0.00 -> 130.1 mm, vias 0 -> 5
- added copper zone on B.Cu, net GND
- added copper zone on F.Cu, net GND
- added copper zone on In2.Cu, net GND
Other:
- net class Default: trace_width 0.254 -> 0.3048
- rule via_min_drill: 0.508 -> 0.5
- board text added: "+12V"
- board text added: "+19V"
- board text added: "+5VD"
- board text added: "+7.5V"
- board text added: "-19V"
- board text added: "-7.5V"
- board text added: "AGND DGND"
- board text added: "DAC A ±5V"
- board text added: "DAC B ±5V"
- board text added: "DAC C ±16.384V"
- board text added: "DAC D ±16.384V"
- board text added: "GND"
- board text added: "GNDA"
