File: MicroFLiC_DAC_1_0.sch (KiCad schematic (older format))
At the start: 34 parts, among them P1 2x4_MicroMaTch, P2 2x4_HEADER, P3 SMA, P4 SMA, P5 SMA, P6 SMA, P7 1x2_HEADER, P8 1x2_SOCKET, U1 DAC8734

Commit message: Final production board v1.0
Parts:
- added A1: JMP, jakub:JMP, symbol JMP
Connections:
- wire segments 195 -> 196
Changed lines of the file:
@@
 EESchema Schematic File Version 2
+LIBS:MicroFLiC_DAC_1_0-rescue
 LIBS:power
 LIBS:device
@@
 $EndComp
 Wire Wire Line
-	3850 1650 3950 1650
+	3750 1650 3950 1650
 Wire Wire Line
 	3950 1550 3950 1750
@@
 	3950 1750 5100 1750
 Wire Wire Line
-	3850 1850 5100 1850
-Wire Wire Line
-	3350 1650 3250 1650
+	3750 1850 5100 1850
+Wire Wire Line
+	3450 1650 3250 1650
 Wire Wire Line
 	3250 1650 3250 2350
 Wire Wire Line
-	3350 1850 3250 1850
+	3450 1850 3250 1850
 Connection ~ 3250 1850
 $Comp
@@
 $EndComp
 Wire Wire Line
-	4550 1500 4550 1650
+	4550 1400 4550 1650
 Wire Wire Line
 	4550 1650 5100 1650
@@
 Connection ~ 4250 850
 Wire Wire Line
-	4550 850  4550 1000
+	4550 850  4550 1100
 $Comp
 L R R3
@@
 $EndComp
 Wire Wire Line
-	3350 2050 3250 2050
+	3450 2050 3250 2050
 Connection ~ 3250 2050
 Wire Wire Line
-	3350 2250 3250 2250
+	3450 2250 3250 2250
 Connection ~ 3250 2250
 Wire Wire Line
-	3850 2050 5100 2050
+	3750 2050 5100 2050
 Wire Wire Line
 	5100 2150 3950 2150
@@
 	3950 2150 3950 2250
 Wire Wire Line
-	3950 2250 3850 2250
+	3950 2250 3750 2250
 $Sheet
 S 8600 1450 1300 800
@@
 $EndComp
 Wire Wire Line
-	2200 6700 2200 6800
-Wire Wire Line
-	2800 6400 2800 6800
+	2200 6700 2200 6850
+Wire Wire Line
+	2800 6400 2800 6850
 Connection ~ 2500 6700
 Wire Wire Line
-	2200 7200 2200 7400
-Wire Wire Line
-	2800 7300 2800 7200
+	2200 7150 2200 7400
+Wire Wire Line
+	2800 7300 2800 7150
 Connection ~ 2500 7300
 $Comp
@@
 $EndComp
 Wire Wire Line
-	4200 7300 4200 7200
-Wire Wire Line
-	4200 6700 4200 6800
-Wire Wire Line
-	3600 6600 3600 6800
-Wire Wire Line
-	3600 7200 3600 7400
+	4200 7300 4200 7150
+Wire Wire Line
+	4200 6700 4200 6850
+Wire Wire Line
+	3600 6600 3600 6850
+Wire Wire Line
+	3600 7150 3600 7400
 $Comp
 L VSS #PWR021
@@
 $EndComp
 Wire Wire Line
-	3250 6400 3300 6400
-Wire Wire Line
-	2800 6400 2850 6400
+	3200 6400 3300 6400
+Wire Wire Line
+	2800 6400 2900 6400
 $Comp
 L C C11
@@
 $EndComp
 Wire Wire Line
-	5600 6700 5600 6800
-Wire Wire Line
-	5600 7300 5600 7200
-Wire Wire Line
-	5300 7300 5300 7200
-Wire Wire Line
-	5300 6800 5300 6700
+	5600 6700 5600 6850
+Wire Wire Line
+	5600 7300 5600 7150
+Wire Wire Line
+	5300 7300 5300 7150
+Wire Wire Line
+	5300 6850 5300 6700
 Wire Wire Line
 	5300 7300 5600 7300
@@
 	1900 7300 2800 7300
 Wire Wire Line
-	3250 6700 4200 6700
-Wire Wire Line
-	1900 6700 2850 6700
+	3200 6700 4200 6700
+Wire Wire Line
+	1900 6700 2900 6700
 $Comp
 L CP2 C3
@@
 L GND #PWR025
 U 1 1 557F06F3
-P 8000 6250
-F 0 "#PWR025" H 8000 6000 60  0001 C CNN
-F 1 "GND" H 8000 6100 60  0000 C CNN
-F 2 "" H 8000 6250 60  0000 C CNN
-F 3 "" H 8000 6250 60  0000 C CNN
-	1    8000 6250
+P 7750 6100
+F 0 "#PWR025" H 7750 5850 60  0001 C CNN
+F 1 "GND" H 7750 5950 60  0000 C CNN
+F 2 "" H 7750 6100 60  0000 C CNN
+F 3 "" H 7750 6100 60  0000 C CNN
+	1    7750 6100
 	1    0    0    -1
 $EndComp
@@
 L GNDA #PWR026
 U 1 1 557F082A
-P 8250 6250
-F 0 "#PWR026" H 8250 6000 60  0001 C CNN
-F 1 "GNDA" H 8250 6100 60  0000 C CNN
-F 2 "" H 8250 6250 60  0000 C CNN
-F 3 "" H 8250 6250 60  0000 C CNN
-	1    8250 6250
-	1    0    0    -1
-$EndComp
-Wire Wire Line
-	8250 6250 8250 6200
-Wire Wire Line
-	8250 6200 8000 6200
-Wire Wire Line
-	8000 6200 8000 6250
+P 8450 6100
+F 0 "#PWR026" H 8450 5850 60  0001 C CNN
+F 1 "GNDA" H 8450 5950 60  0000 C CNN
+F 2 "" H 8450 6100 60  0000 C CNN
+F 3 "" H 8450 6100 60  0000 C CNN
+	1    8450 6100
+	1    0    0    -1
+$EndComp
+Wire Wire Line
+	8450 6100 8450 6000
+Wire Wire Line
+	7750 6000 7750 6100
 $Comp
 L CONN_02X04 P2
@@
 Text Label 4950 6050 0    60   ~ 0
 -7.5V
+$Comp
+L JMP A1
+U 1 1 566887AB
+P 8100 6000
+F 0 "A1" H 8100 6150 60  0000 C CNN
+F 1 "JMP" H 8100 5850 60  0000 C CNN
+F 2 "jakub:JMP" H 8100 6000 60  0001 C CNN
+F 3 "" H 8100 6000 60  0000 C CNN
+	1    8100 6000
+	1    0    0    -1
+$EndComp
+Wire Wire Line
+	8450 6000 8400 6000
+Wire Wire Line
+	7800 6000 7750 6000
 $EndSCHEMATC
