File: digitalIsolation_1_0.sch (KiCad schematic (older format))
At the start: 6 parts, among them U14 74AHC1G14, U15 Si8651

Commit message: Final production board v1.0
Changed lines of the file:
@@
 EESchema Schematic File Version 2
+LIBS:MicroFLiC_DAC_1_0-rescue
 LIBS:power
 LIBS:device
@@
 U 1 1 5574AB6E
 P 8100 3500
+AR Path="/5574AB6E" Ref="C67"  Part="1"
+AR Path="/5574A638/5574AB6E" Ref="C67"  Part="1"
 F 0 "C67" H 8150 3600 50  0000 L CNN
 F 1 "100n" H 8150 3400 50  0000 L CNN
@@
 $EndComp
 Wire Wire Line
-	8100 3100 8100 3300
+	8100 3100 8100 3350
 Connection ~ 7800 3200
 $Comp
@@
 	7800 3500 7800 3800
 Wire Wire Line
-	8100 3700 8100 3800
+	8100 3650 8100 3800
 $Comp
 L GND #PWR084
@@
 U 1 1 5574AE37
 P 6000 3500
+AR Path="/5574AE37" Ref="C66"  Part="1"
+AR Path="/5574A638/5574AE37" Ref="C66"  Part="1"
 F 0 "C66" H 6050 3600 50  0000 L CNN
 F 1 "100n" H 6050 3400 50  0000 L CNN
@@
 	6000 3200 6400 3200
 Wire Wire Line
-	6000 2900 6000 3300
-Wire Wire Line
-	6000 3800 6000 3700
+	6000 2900 6000 3350
+Wire Wire Line
+	6000 3800 6000 3650
 Wire Wire Line
 	6400 3500 6300 3500
@@
 U 1 1 5574AD7F
 P 4300 3500
+AR Path="/5574AD7F" Ref="C65"  Part="1"
+AR Path="/5574A638/5574AD7F" Ref="C65"  Part="1"
 F 0 "C65" H 4350 3600 50  0000 L CNN
 F 1 "100n" H 4350 3400 50  0000 L CNN
@@
 	5200 2900 5200 3000
 Wire Wire Line
-	4300 2900 4300 3300
+	4300 2900 4300 3350
 Connection ~ 5200 2900
 Wire Wire Line
-	4300 3700 4300 3800
+	4300 3650 4300 3800
 Wire Wire Line
 	6300 3800 3600 3800
@@
 Connection ~ 4700 2200
 Wire Wire Line
-	4300 3200 3600 3200
+	3600 3200 4300 3200
 Connection ~ 4300 3200
 Connection ~ 4300 3800
@@
 U 1 1 5574B7E4
 P 4000 3500
+AR Path="/5574B7E4" Ref="C64"  Part="1"
+AR Path="/5574A638/5574B7E4" Ref="C64"  Part="1"
 F 0 "C64" H 4050 3600 50  0000 L CNN
 F 1 "10u" H 4050 3400 50  0000 L CNN
@@
 $EndComp
 Wire Wire Line
-	4000 3300 4000 3200
+	4000 3350 4000 3200
 Connection ~ 4000 3200
 Wire Wire Line
-	4000 3700 4000 3800
+	4000 3650 4000 3800
 Connection ~ 4000 3800
 $EndSCHEMATC
