File: powerSupply_1_0.sch (KiCad schematic (older format))
At the start: 40 parts, among them U10 TPS7A4901, U11 LM3880, U12 TPS7A3001, U13 TPS7A3001, U8 TPS7A4901, U9 TPS7A4901

Commit message: Final production board v1.0
Connections:
- net labels removed: GND

Commit message: Updated part names
Parts:
- C43, C52, C55, C62: value 4u7 -> 4u7/25V; Alt. Order Code (none) -> 81-GRM21BR61E475MA2L; Alt. Supplier (none) -> Mouser; Note (none) -> 4μ7/25V X5R 0805 ceramic capacitor; Package (none) -> 0805; Part Number GRM21BR61E475KA12L -> GRM21BR61E475MA12L; Supplier (none) -> Farnell
Connections:
- wire segments 142 -> 181
Other:
- moved on the sheet: C43
