File: MicroFLiC_DAC.sch (KiCad schematic (older format))
At the start: 33 parts, among them P1 8-way Micro-MaTch, P2 2x4 header strip, P3 1x2 header strip, P4 1x2 socket strip, P5 SMA, P6 SMA, P7 SMA, P8 SMA, U1 DAC8734

Commit message: Fixed can, 1Ohm resistor descriptions
Parts:
- removed A1: JMP, jakub:solder_jumper, symbol JMP
- added JP7: GND/GNDA, jakub:solder_jumper, symbol JUMPER
- S1, S2: footprint jakub:can-MS323-20 -> jakub:can-MS257-10; Alt. Order Code MS323-20 -> MS257-10; Order Code 826-6788 -> 826-6766; Part Number MS323-20 -> MS257-10
Connections:
- wire segments 194 -> 196
Other:
- note added: "Solder bridge\nor ferrite bead"
- moved on the sheet: S1, S2
Changed lines of the file:
@@
 	5300 7300 5300 7150
-Wire Wire Line
-	5300 6850 5300 6700
 Wire Wire Line
 	5300 7300 5600 7300
@@
 $EndComp
 Wire Wire Line
-	5300 5050 4450 5050
+	4450 5050 5300 5050
 Wire Wire Line
 	4450 5050 4450 5300
@@
 Wire Wire Line
 	4300 5200 4300 5950
-Wire Wire Line
-	4300 5950 4550 5950
 Wire Wire Line
 	4550 5800 4550 6150
@@
 L GND #PWR025
 U 1 1 557F06F3
-P 7750 6100
-F 0 "#PWR025" H 7750 5850 60  0001 C CNN
-F 1 "GND" H 7750 5950 60  0000 C CNN
-F 2 "" H 7750 6100 60  0000 C CNN
-F 3 "" H 7750 6100 60  0000 C CNN
-	1    7750 6100
+P 7800 6100
+F 0 "#PWR025" H 7800 5850 60  0001 C CNN
+F 1 "GND" H 7800 5950 60  0000 C CNN
+F 2 "" H 7800 6100 60  0000 C CNN
+F 3 "" H 7800 6100 60  0000 C CNN
+	1    7800 6100
 	1    0    0    -1
 $EndComp
@@
 L GNDA #PWR026
 U 1 1 557F082A
-P 8450 6100
-F 0 "#PWR026" H 8450 5850 60  0001 C CNN
-F 1 "GNDA" H 8450 5950 60  0000 C CNN
-F 2 "" H 8450 6100 60  0000 C CNN
-F 3 "" H 8450 6100 60  0000 C CNN
-	1    8450 6100
-	1    0    0    -1
-$EndComp
-Wire Wire Line
-	8450 6100 8450 6000
-Wire Wire Line
-	7750 6000 7750 6100
+P 8500 6100
+F 0 "#PWR026" H 8500 5850 60  0001 C CNN
+F 1 "GNDA" H 8500 5950 60  0000 C CNN
+F 2 "" H 8500 6100 60  0000 C CNN
+F 3 "" H 8500 6100 60  0000 C CNN
+	1    8500 6100
+	1    0    0    -1
+$EndComp
+Wire Wire Line
+	8500 5900 8500 6100
+Wire Wire Line
+	7800 5900 7800 6100
 $Comp
 L CONN_02X04 P2
@@
 $EndComp
 Wire Wire Line
-	4750 5300 4750 4950
+	4750 4700 4750 5300
 $Comp
 L +5VD #PWR028
 U 1 1 557F25CE
-P 4750 4950
-F 0 "#PWR028" H 4750 4800 60  0001 C CNN
-F 1 "+5VD" H 4750 5090 60  0000 C CNN
-F 2 "" H 4750 4950 60  0000 C CNN
-F 3 "" H 4750 4950 60  0000 C CNN
-	1    4750 4950
+P 4750 4700
+F 0 "#PWR028" H 4750 4550 60  0001 C CNN
+F 1 "+5VD" H 4750 4840 60  0000 C CNN
+F 2 "" H 4750 4700 60  0000 C CNN
+F 3 "" H 4750 4700 60  0000 C CNN
+	1    4750 4700
 	1    0    0    -1
 $EndComp
@@
 L CONN_01X02 S2
 U 1 1 557F4470
-P 9200 5950
-F 0 "S2" H 9200 6100 50  0000 C CNN
-F 1 "shield_can" V 9300 5950 50  0000 C CNN
-F 2 "jakub:can-MS323-20" H 9200 5950 60  0001 C CNN
-F 3 "" H 9200 5950 60  0000 C CNN
-F 4 "MS323-20" H 9200 5950 60  0001 C CNN "Part Number"
-F 5 "Masach" H 9200 5950 60  0001 C CNN "Manufacturer"
-F 6 "Can" H 9200 5950 60  0001 C CNN "Package"
-F 7 "RS Components" H 9200 5950 60  0001 C CNN "Supplier"
-F 8 "826-6788" H 9200 5950 60  0001 C CNN "Order Code"
-F 9 "Masach" H 9200 5950 60  0001 C CNN "Alt. Supplier"
-F 10 "MS323-20" H 9200 5950 60  0001 C CNN "Alt. Order Code"
-F 11 "Two-piece EMI shielding can" H 9200 5950 60  0001 C CNN "Note"
-	1    9200 5950
-	1    0    0    -1
-$EndComp
-Wire Wire Line
-	8900 6000 8900 6100
-Wire Wire Line
-	8900 6000 9000 6000
-Connection ~ 8900 6000
+P 9400 5950
+F 0 "S2" H 9400 6100 50  0000 C CNN
+F 1 "shield_can" V 9500 5950 50  0000 C CNN
+F 2 "jakub:can-MS257-10" H 9400 5950 60  0001 C CNN
+F 3 "" H 9400 5950 60  0000 C CNN
+F 4 "MS257-10" H 9400 5950 60  0001 C CNN "Part Number"
+F 5 "Masach" H 9400 5950 60  0001 C CNN "Manufacturer"
+F 6 "Can" H 9400 5950 60  0001 C CNN "Package"
+F 7 "RS Components" H 9400 5950 60  0001 C CNN "Supplier"
+F 8 "826-6766" H 9400 5950 60  0001 C CNN "Order Code"
+F 9 "Masach" H 9400 5950 60  0001 C CNN "Alt. Supplier"
+F 10 "MS257-10" H 9400 5950 60  0001 C CNN "Alt. Order Code"
+F 11 "Two-piece EMI shielding can" H 9400 5950 60  0001 C CNN "Note"
+	1    9400 5950
+	1    0    0    -1
+$EndComp
+Wire Wire Line
+	9100 6000 9100 6100
+Wire Wire Line
+	9100 6000 9200 6000
 $Comp
 L GNDA #PWR029
 U 1 1 557F4631
-P 8900 6100
-F 0 "#PWR029" H 8900 5850 60  0001 C CNN
-F 1 "GNDA" H 8900 5950 60  0000 C CNN
-F 2 "" H 8900 6100 60  0000 C CNN
-F 3 "" H 8900 6100 60  0000 C CNN
-	1    8900 6100
+P 9100 6100
+F 0 "#PWR029" H 9100 5850 60  0001 C CNN
+F 1 "GNDA" H 9100 5950 60  0000 C CNN
+F 2 "" H 9100 6100 60  0000 C CNN
+F 3 "" H 9100 6100 60  0000 C CNN
+	1    9100 6100
 	1    0    0    -1
 $EndComp
@@
 L CONN_01X02 S1
 U 1 1 55808F86
-P 9200 5400
-F 0 "S1" H 9200 5550 50  0000 C CNN
-F 1 "shield_can" V 9300 5400 50  0000 C CNN
-F 2 "jakub:can-MS323-20" H 9200 5400 60  0001 C CNN
-F 3 "" H 9200 5400 60  0000 C CNN
-F 4 "MS323-20" H 9200 5400 60  0001 C CNN "Part Number"
-F 5 "Masach" H 9200 5400 60  0001 C CNN "Manufacturer"
-F 6 "Can" H 9200 5400 60  0001 C CNN "Package"
-F 7 "RS Components" H 9200 5400 60  0001 C CNN "Supplier"
-F 8 "826-6788" H 9200 5400 60  0001 C CNN "Order Code"
-F 9 "Masach" H 9200 5400 60  0001 C CNN "Alt. Supplier"
-F 10 "MS323-20" H 9200 5400 60  0001 C CNN "Alt. Order Code"
-F 11 "Two-piece EMI shielding can" H 9200 5400 60  0001 C CNN "Note"
-	1    9200 5400
-	1    0    0    -1
-$EndComp
-Wire Wire Line
-	9000 5350 8900 5350
-Wire Wire Line
-	8900 5350 8900 5550
+P 9400 5350
+F 0 "S1" H 9400 5500 50  0000 C CNN
+F 1 "shield_can" V 9500 5350 50  0000 C CNN
+F 2 "jakub:can-MS257-10" H 9400 5350 60  0001 C CNN
+F 3 "" H 9400 5350 60  0000 C CNN
+F 4 "MS257-10" H 9400 5350 60  0001 C CNN "Part Number"
+F 5 "Masach" H 9400 5350 60  0001 C CNN "Manufacturer"
+F 6 "Can" H 9400 5350 60  0001 C CNN "Package"
+F 7 "RS Components" H 9400 5350 60  0001 C CNN "Supplier"
+F 8 "826-6766" H 9400 5350 60  0001 C CNN "Order Code"
+F 9 "Masach" H 9400 5350 60  0001 C CNN "Alt. Supplier"
+F 10 "MS257-10" H 9400 5350 60  0001 C CNN "Alt. Order Code"
+F 11 "Two-piece EMI shielding can" H 9400 5350 60  0001 C CNN "Note"
+	1    9400 5350
+	1    0    0    -1
+$EndComp
+Wire Wire Line
+	9200 5300 9100 5300
+Wire Wire Line
+	9100 5300 9100 5500
 $Comp
 L GNDA #PWR030
 U 1 1 55808F90
-P 8900 5550
-F 0 "#PWR030" H 8900 5300 60  0001 C CNN
-F 1 "GNDA" H 8900 5400 60  0000 C CNN
-F 2 "" H 8900 5550 60  0000 C CNN
-F 3 "" H 8900 5550 60  0000 C CNN
-	1    8900 5550
+P 9100 5500
+F 0 "#PWR030" H 9100 5250 60  0001 C CNN
+F 1 "GNDA" H 9100 5350 60  0000 C CNN
+F 2 "" H 9100 5500 60  0000 C CNN
+F 3 "" H 9100 5500 60  0000 C CNN
+	1    9100 5500
 	1    0    0    -1
 $EndComp
@@
 Text Label 4950 6050 0    60   ~ 0
 -7.5V
-$Comp
-L JMP A1
-U 1 1 566887AB
-P 8100 6000
-F 0 "A1" H 8100 6150 60  0000 C CNN
-F 1 "JMP" H 8100 5850 60  0000 C CNN
-F 2 "jakub:solder_jumper" H 8100 6000 60  0001 C CNN
-F 3 "" H 8100 6000 60  0000 C CNN
-	1    8100 6000
-	1    0    0    -1
-$EndComp
-Wire Wire Line
-	8450 6000 8400 6000
-Wire Wire Line
-	7800 6000 7750 6000
+Wire Wire Line
+	8500 6000 8450 6000
+Wire Wire Line
+	7850 6000 7800 6000
 Connection ~ 8000 2050
 Connection ~ 8000 3250
@@
 NoConn ~ 5100 2050
 NoConn ~ 5100 2150
-NoConn ~ 9000 5900
-NoConn ~ 9000 5450
+NoConn ~ 9200 5900
+NoConn ~ 9200 5400
+Wire Wire Line
+	5300 6850 5300 6700
+Wire Wire Line
+	4750 4800 4400 4800
+Wire Wire Line
+	4400 4800 4400 4700
+Connection ~ 4750 4800
+$Comp
+L PWR_FLAG #FLG031
+U 1 1 56F28740
+P 4400 4700
+F 0 "#FLG031" H 4400 4795 50  0001 C CNN
+F 1 "PWR_FLAG" H 4400 4880 50  0000 C CNN
+F 2 "" H 4400 4700 50  0000 C CNN
+F 3 "" H 4400 4700 50  0000 C CNN
+	1    4400 4700
+	1    0    0    -1
+$EndComp
+$Comp
+L PWR_FLAG #FLG032
+U 1 1 56F28B4E
+P 7800 5900
+F 0 "#FLG032" H 7800 5995 50  0001 C CNN
+F 1 "PWR_FLAG" H 7800 6080 50  0000 C CNN
+F 2 "" H 7800 5900 50  0000 C CNN
+F 3 "" H 7800 5900 50  0000 C CNN
+	1    7800 5900
+	1    0    0    -1
+$EndComp
+Wire Wire Line
+	4300 5950 4550 5950
+$Comp
+L PWR_FLAG #FLG033
+U 1 1 56F2F7DE
+P 8500 5900
+F 0 "#FLG033" H 8500 5995 50  0001 C CNN
+F 1 "PWR_FLAG" H 8500 6080 50  0000 C CNN
+F 2 "" H 8500 5900 50  0000 C CNN
+F 3 "" H 8500 5900 50  0000 C CNN
+	1    8500 5900
+	1    0    0    -1
+$EndComp
+Connection ~ 8500 6000
+Connection ~ 7800 6000
+$Comp
+L JUMPER JP7
+U 1 1 56F1D54A
+P 8150 6000
+F 0 "JP7" H 8150 6150 50  0000 C CNN
+F 1 "GND/GNDA" H 8150 5920 50  0000 C CNN
+F 2 "jakub:solder_jumper" H 8150 6000 60  0001 C CNN
+F 3 "" H 8150 6000 60  0000 C CNN
+	1    8150 6000
+	1    0    0    -1
+$EndComp
+Text Notes 7800 5600 0    60   ~ 0
+Solder bridge\nor ferrite bead
 $EndSCHEMATC

Commit message: Finalized PCB for production
Parts:
- C10, C11, C2, C4, C8: Alt. Order Code 710-885012206095 -> 603-CC603KRX7R9BB104; Manufacturer Multicomp -> Yageo; Order Code 1759122 -> 1362556; Part Number MC0603B104K500CT -> CC0603KRX7R9BB104
- C5, C6: Alt. Order Code 77-VJ0603Y103KXACBC -> 603-CC603KRX7R9BB103; Manufacturer Multicomp -> Yageo; Note 10nF/100V X7R 0603 ceramic capacitor -> 10nF/50V X7R 0603 ceramic capacitor; Order Code 2320786 -> 722236; Part Number MC0603B103K101CT -> CC0603KRX7R9BB103
- R1, R2, R3: value 10k -> 12k; footprint Resistors_SMD:R_0805 -> Resistors_SMD:R_0603; Alt. Order Code 71-CRCW0805-10K-E3 -> 603-RC0603FR-0712KL; Manufacturer Multicomp -> Yageo; Order Code 2073607 -> 9238611; Package 0805 -> 0603; Part Number MCMR08X1002FTL -> RC0603FR-0712KL
