File: highCurrentAmp.sch (KiCad schematic (older format))
At the start: 20 parts, among them U4 AD8021, U5 AD8021

Commit message: Fixed can, 1Ohm resistor descriptions
Parts:
- C32, C34, C40, C42: value 470p -> 10n; Alt. Order Code 710-885012206081 -> 77-VJ0603Y103KXACBC; Note 470pF/50V C0G(NP0) 0603 ceramic capacitor -> 10nF/100V X7R 0603 ceramic capacitor; Order Code 1759080 -> 2320786; Part Number MC0603N471J500CT -> MC0603B103K101CT
Changed lines of the file:
@@
 $EndDescr
-$Comp
-L C C32
-U 1 1 55742E4A
-P 3550 2100
-F 0 "C32" H 3600 2200 50  0000 L CNN
-F 1 "470p" H 3600 2000 50  0000 L CNN
-F 2 "Capacitors_SMD:C_0603" H 3588 1950 30  0001 C CNN
-F 3 "" H 3550 2100 60  0000 C CNN
-F 4 "MC0603N471J500CT" H 3550 2100 60  0001 C CNN "Part Number"
-F 5 "Multicomp" H 3550 2100 60  0001 C CNN "Manufacturer"
-F 6 "0603" H 3550 2100 60  0001 C CNN "Package"
-F 7 "Farnell" H 3550 2100 60  0001 C CNN "Supplier"
-F 8 "1759080" H 3550 2100 60  0001 C CNN "Order Code"
-F 9 "Mouser" H 3550 2100 60  0001 C CNN "Alt. Supplier"
-F 10 "710-885012206081" H 3550 2100 60  0001 C CNN "Alt. Order Code"
-F 11 "470pF/50V C0G(NP0) 0603 ceramic capacitor" H 3550 2100 60  0001 C CNN "Note"
-	1    3550 2100
-	0    1    1    0
-$EndComp
 $Comp
 L C C31
@@
 $EndComp
 $Comp
-L C C34
-U 1 1 55733A48
-P 3600 3400
-F 0 "C34" H 3650 3500 50  0000 L CNN
-F 1 "470p" H 3650 3300 50  0000 L CNN
-F 2 "Capacitors_SMD:C_0603" H 3638 3250 30  0001 C CNN
-F 3 "" H 3600 3400 60  0000 C CNN
-F 4 "MC0603N471J500CT" H 3550 2250 60  0001 C CNN "Part Number"
-F 5 "Multicomp" H 3550 2250 60  0001 C CNN "Manufacturer"
-F 6 "0603" H 3600 3400 60  0001 C CNN "Package"
-F 7 "Farnell" H 3600 3400 60  0001 C CNN "Supplier"
-F 8 "1759080" H 3550 2250 60  0001 C CNN "Order Code"
-F 9 "Mouser" H 3600 3400 60  0001 C CNN "Alt. Supplier"
-F 10 "710-885012206081" H 3600 3400 60  0001 C CNN "Alt. Order Code"
-F 11 "470pF/50V C0G(NP0) 0603 ceramic capacitor" H 3600 3400 60  0001 C CNN "Note"
-	1    3600 3400
-	0    1    1    0
-$EndComp
-$Comp
 L C C35
 U 1 1 55742E4D
@@
 $EndComp
 $Comp
-L GNDA #PWR039
+L GNDA #PWR042
 U 1 1 55742E4E
 P 3850 2200
-F 0 "#PWR039" H 3850 1950 60  0001 C CNN
+F 0 "#PWR042" H 3850 1950 60  0001 C CNN
 F 1 "GNDA" H 3850 2050 60  0000 C CNN
 F 2 "" H 3850 2200 60  0000 C CNN
@@
 $EndComp
 $Comp
-L GNDA #PWR040
+L GNDA #PWR043
 U 1 1 55742E4F
 P 3900 4100
-F 0 "#PWR040" H 3900 3850 60  0001 C CNN
+F 0 "#PWR043" H 3900 3850 60  0001 C CNN
 F 1 "GNDA" H 3900 3950 60  0000 C CNN
 F 2 "" H 3900 4100 60  0000 C CNN
@@
 $EndComp
 $Comp
-L C C40
-U 1 1 55742E51
-P 8150 2100
-F 0 "C40" H 8200 2200 50  0000 L CNN
-F 1 "470p" H 8200 2000 50  0000 L CNN
-F 2 "Capacitors_SMD:C_0603" H 8188 1950 30  0001 C CNN
-F 3 "" H 8150 2100 60  0000 C CNN
-F 4 "MC0603N471J500CT" H 3550 2100 60  0001 C CNN "Part Number"
-F 5 "Multicomp" H 3550 2100 60  0001 C CNN "Manufacturer"
-F 6 "0603" H 8150 2100 60  0001 C CNN "Package"
-F 7 "Farnell" H 8150 2100 60  0001 C CNN "Supplier"
-F 8 "1759080" H 3550 2100 60  0001 C CNN "Order Code"
-F 9 "Mouser" H 8150 2100 60  0001 C CNN "Alt. Supplier"
-F 10 "710-885012206081" H 8150 2100 60  0001 C CNN "Alt. Order Code"
-F 11 "470pF/50V C0G(NP0) 0603 ceramic capacitor" H 8150 2100 60  0001 C CNN "Note"
-	1    8150 2100
-	0    1    1    0
-$EndComp
-$Comp
 L C C39
 U 1 1 55742E52
@@
 $EndComp
 $Comp
-L C C42
-U 1 1 55742E53
-P 8200 3400
-F 0 "C42" H 8250 3500 50  0000 L CNN
-F 1 "470p" H 8250 3300 50  0000 L CNN
-F 2 "Capacitors_SMD:C_0603" H 8238 3250 30  0001 C CNN
-F 3 "" H 8200 3400 60  0000 C CNN
-F 4 "MC0603N471J500CT" H 3550 2250 60  0001 C CNN "Part Number"
-F 5 "Multicomp" H 3550 2250 60  0001 C CNN "Manufacturer"
-F 6 "0603" H 8200 3400 60  0001 C CNN "Package"
-F 7 "Farnell" H 8200 3400 60  0001 C CNN "Supplier"
-F 8 "1759080" H 3550 2250 60  0001 C CNN "Order Code"
-F 9 "Mouser" H 8200 3400 60  0001 C CNN "Alt. Supplier"
-F 10 "710-885012206081" H 8200 3400 60  0001 C CNN "Alt. Order Code"
-F 11 "470pF/50V C0G(NP0) 0603 ceramic capacitor" H 8200 3400 60  0001 C CNN "Note"
-	1    8200 3400
-	0    1    1    0
-$EndComp
-$Comp
 L C C43
 U 1 1 55742E54
@@
 $EndComp
 $Comp
-L GNDA #PWR041
+L GNDA #PWR044
 U 1 1 55742E55
 P 8450 2200
-F 0 "#PWR041" H 8450 1950 60  0001 C CNN
+F 0 "#PWR044" H 8450 1950 60  0001 C CNN
 F 1 "GNDA" H 8450 2050 60  0000 C CNN
 F 2 "" H 8450 2200 60  0000 C CNN
@@
 $EndComp
 $Comp
-L GNDA #PWR042
+L GNDA #PWR045
 U 1 1 557342A6
 P 8500 4100
-F 0 "#PWR042" H 8500 3850 60  0001 C CNN
+F 0 "#PWR045" H 8500 3850 60  0001 C CNN
 F 1 "GNDA" H 8500 3950 60  0000 C CNN
 F 2 "" H 8500 4100 60  0000 C CNN
@@
 $EndComp
 $Comp
-L +6V #PWR043
+L +6V #PWR046
 U 1 1 55738BED
 P 3100 1800
-F 0 "#PWR043" H 3100 1650 60  0001 C CNN
+F 0 "#PWR046" H 3100 1650 60  0001 C CNN
 F 1 "+6V" H 3100 1940 60  0000 C CNN
 F 2 "" H 3100 1800 60  0000 C CNN
@@
 $EndComp
 $Comp
-L +6V #PWR044
+L +6V #PWR047
 U 1 1 56E01424
 P 7700 1800
-F 0 "#PWR044" H 7700 1650 60  0001 C CNN
+F 0 "#PWR047" H 7700 1650 60  0001 C CNN
 F 1 "+6V" H 7700 1940 60  0000 C CNN
 F 2 "" H 7700 1800 60  0000 C CNN
@@
 	8450 1350 8300 1350
 Connection ~ 8450 1800
+$Comp
+L C C32
+U 1 1 56F15165
+P 3550 2100
+F 0 "C32" H 3600 2200 50  0000 L CNN
+F 1 "10n" H 3600 2000 50  0000 L CNN
+F 2 "Capacitors_SMD:C_0603" H 3588 1950 30  0001 C CNN
+F 3 "" H 3550 2100 60  0000 C CNN
+F 4 "MC0603B103K101CT" H 3550 2100 60  0001 C CNN "Part Number"
+F 5 "Multicomp" H 3550 2100 60  0001 C CNN "Manufacturer"
+F 6 "0603" H 3550 2100 60  0001 C CNN "Package"
+F 7 "Farnell" H 3550 2100 60  0001 C CNN "Supplier"
+F 8 "2320786" H 3550 2100 60  0001 C CNN "Order Code"
+F 9 "Mouser" H 3550 2100 60  0001 C CNN "Alt. Supplier"
+F 10 "77-VJ0603Y103KXACBC" H 3550 2100 60  0001 C CNN "Alt. Order Code"
+F 11 "10nF/100V X7R 0603 ceramic capacitor" H 3550 2100 60  0001 C CNN "Note"
+	1    3550 2100
+	0    1    1    0
+$EndComp
+$Comp
+L C C34
+U 1 1 56F152BD
+P 3600 3400
+F 0 "C34" H 3650 3500 50  0000 L CNN
+F 1 "10n" H 3650 3300 50  0000 L CNN
+F 2 "Capacitors_SMD:C_0603" H 3638 3250 30  0001 C CNN
+F 3 "" H 3600 3400 60  0000 C CNN
+F 4 "MC0603B103K101CT" H 3600 3400 60  0001 C CNN "Part Number"
+F 5 "Multicomp" H 3600 3400 60  0001 C CNN "Manufacturer"
+F 6 "0603" H 3600 3400 60  0001 C CNN "Package"
+F 7 "Farnell" H 3600 3400 60  0001 C CNN "Supplier"
+F 8 "2320786" H 3600 3400 60  0001 C CNN "Order Code"
+F 9 "Mouser" H 3600 3400 60  0001 C CNN "Alt. Supplier"
+F 10 "77-VJ0603Y103KXACBC" H 3600 3400 60  0001 C CNN "Alt. Order Code"
+F 11 "10nF/100V X7R 0603 ceramic capacitor" H 3600 3400 60  0001 C CNN "Note"
+	1    3600 3400
+	0    1    1    0
+$EndComp
+$Comp
+L C C40
+U 1 1 56F154AB
+P 8150 2100
+F 0 "C40" H 8200 2200 50  0000 L CNN
+F 1 "10n" H 8200 2000 50  0000 L CNN
+F 2 "Capacitors_SMD:C_0603" H 8188 1950 30  0001 C CNN
+F 3 "" H 8150 2100 60  0000 C CNN
+F 4 "MC0603B103K101CT" H 8150 2100 60  0001 C CNN "Part Number"
+F 5 "Multicomp" H 8150 2100 60  0001 C CNN "Manufacturer"
+F 6 "0603" H 8150 2100 60  0001 C CNN "Package"
+F 7 "Farnell" H 8150 2100 60  0001 C CNN "Supplier"
+F 8 "2320786" H 8150 2100 60  0001 C CNN "Order Code"
+F 9 "Mouser" H 8150 2100 60  0001 C CNN "Alt. Supplier"
+F 10 "77-VJ0603Y103KXACBC" H 8150 2100 60  0001 C CNN "Alt. Order Code"
+F 11 "10nF/100V X7R 0603 ceramic capacitor" H 8150 2100 60  0001 C CNN "Note"
+	1    8150 2100
+	0    1    1    0
+$EndComp
+$Comp
+L C C42
+U 1 1 56F155A0
+P 8200 3400
+F 0 "C42" H 8250 3500 50  0000 L CNN
+F 1 "10n" H 8250 3300 50  0000 L CNN
+F 2 "Capacitors_SMD:C_0603" H 8238 3250 30  0001 C CNN
+F 3 "" H 8200 3400 60  0000 C CNN
+F 4 "MC0603B103K101CT" H 8200 3400 60  0001 C CNN "Part Number"
+F 5 "Multicomp" H 8200 3400 60  0001 C CNN "Manufacturer"
+F 6 "0603" H 8200 3400 60  0001 C CNN "Package"
+F 7 "Farnell" H 8200 3400 60  0001 C CNN "Supplier"
+F 8 "2320786" H 8200 3400 60  0001 C CNN "Order Code"
+F 9 "Mouser" H 8200 3400 60  0001 C CNN "Alt. Supplier"
+F 10 "77-VJ0603Y103KXACBC" H 8200 3400 60  0001 C CNN "Alt. Order Code"
+F 11 "10nF/100V X7R 0603 ceramic capacitor" H 8200 3400 60  0001 C CNN "Note"
+	1    8200 3400
+	0    1    1    0
+$EndComp
 $EndSCHEMATC

Commit message: Finalized PCB for production
Parts:
- C29, C32, C34, C37, C40, C42: Alt. Order Code 77-VJ0603Y103KXACBC -> 603-CC603KRX7R9BB103; Manufacturer Multicomp -> Yageo; Note 10nF/100V X7R 0603 ceramic capacitor -> 10nF/50V X7R 0603 ceramic capacitor; Order Code 2320786 -> 722236; Part Number MC0603B103K101CT -> CC0603KRX7R9BB103
- C31, C35, C39, C43: Alt. Order Code 710-885012206095 -> 603-CC603KRX7R9BB104; Manufacturer Multicomp -> Yageo; Order Code 1759122 -> 1362556; Part Number MC0603B104K500CT -> CC0603KRX7R9BB104
- C33, C41: Alt. Order Code 77-VJ0603A100JXACBC -> 603-C0603JRNPO9BN100; Manufacturer Multicomp -> Yageo; Order Code 2320799 -> 721967; Part Number MC0603N100J500CT -> CC0603JRNPO9BN100
