File: reference.sch (KiCad schematic (older format))
At the start: 10 parts, among them U6 REF5040, U7 REF5050

Commit message: Fixed can, 1Ohm resistor descriptions
Parts:
- R10, R11: Alt. Order Code (none) -> 667-ERJ-6GEYJ1R0V; Alt. Supplier (none) -> Mouser; Manufacturer (none) -> Multicomp; Note (none) -> 1Ω/1% 0805 resistor; Order Code (none) -> 2447598; Package (none) -> 0805; Part Number (none) -> MCWR08W1R00FTL; Supplier (none) -> Farnell
Changed lines of the file:
@@
 	2900 2000 2900 2600
 $Comp
-L GNDA #PWR045
+L GNDA #PWR048
 U 1 1 5573B9A8
 P 2900 3000
-F 0 "#PWR045" H 2900 2750 60  0001 C CNN
+F 0 "#PWR048" H 2900 2750 60  0001 C CNN
 F 1 "GNDA" H 2900 2850 60  0000 C CNN
 F 2 "" H 2900 3000 60  0000 C CNN
@@
 $EndComp
 $Comp
-L GNDA #PWR046
+L GNDA #PWR049
 U 1 1 5573B9AE
 P 4900 3000
-F 0 "#PWR046" H 4900 2750 60  0001 C CNN
+F 0 "#PWR049" H 4900 2750 60  0001 C CNN
 F 1 "GNDA" H 4900 2850 60  0000 C CNN
 F 2 "" H 4900 3000 60  0000 C CNN
@@
 	2900 3000 2900 2900
 $Comp
-L GNDA #PWR047
+L GNDA #PWR050
 U 1 1 5573B9C2
 P 5300 3000
-F 0 "#PWR047" H 5300 2750 60  0001 C CNN
+F 0 "#PWR050" H 5300 2750 60  0001 C CNN
 F 1 "GNDA" H 5300 2850 60  0000 C CNN
 F 2 "" H 5300 3000 60  0000 C CNN
@@
 	2900 4100 2900 4700
 $Comp
-L GNDA #PWR048
+L GNDA #PWR051
 U 1 1 5573BE5B
 P 2900 5100
-F 0 "#PWR048" H 2900 4850 60  0001 C CNN
+F 0 "#PWR051" H 2900 4850 60  0001 C CNN
 F 1 "GNDA" H 2900 4950 60  0000 C CNN
 F 2 "" H 2900 5100 60  0000 C CNN
@@
 $EndComp
 $Comp
-L GNDA #PWR049
+L GNDA #PWR052
 U 1 1 5573BE61
 P 4900 5100
-F 0 "#PWR049" H 4900 4850 60  0001 C CNN
+F 0 "#PWR052" H 4900 4850 60  0001 C CNN
 F 1 "GNDA" H 4900 4950 60  0000 C CNN
 F 2 "" H 4900 5100 60  0000 C CNN
@@
 	2900 5100 2900 5000
 $Comp
-L GNDA #PWR050
+L GNDA #PWR053
 U 1 1 5573BE72
 P 5300 5100
-F 0 "#PWR050" H 5300 4850 60  0001 C CNN
+F 0 "#PWR053" H 5300 4850 60  0001 C CNN
 F 1 "GNDA" H 5300 4950 60  0000 C CNN
 F 2 "" H 5300 5100 60  0000 C CNN
@@
 	3400 2600 3400 3400
 $Comp
-L GNDA #PWR051
+L GNDA #PWR054
 U 1 1 5573C48B
 P 3400 3400
-F 0 "#PWR051" H 3400 3150 60  0001 C CNN
+F 0 "#PWR054" H 3400 3150 60  0001 C CNN
 F 1 "GNDA" H 3400 3250 60  0000 C CNN
 F 2 "" H 3400 3400 60  0000 C CNN
@@
 	3400 4700 3400 5500
 $Comp
-L GNDA #PWR052
+L GNDA #PWR055
 U 1 1 5573C579
 P 3400 5500
-F 0 "#PWR052" H 3400 5250 60  0001 C CNN
+F 0 "#PWR055" H 3400 5250 60  0001 C CNN
 F 1 "GNDA" H 3400 5350 60  0000 C CNN
 F 2 "" H 3400 5500 60  0000 C CNN
@@
 F 2 "Resistors_SMD:R_0805" V 5230 2300 50  0001 C CNN
 F 3 "" H 5300 2300 50  0000 C CNN
+F 4 "MCWR08W1R00FTL" H 5300 2300 60  0001 C CNN "Part Number"
+F 5 "Multicomp" H 5300 2300 60  0001 C CNN "Manufacturer"
+F 6 "0805" H 5300 2300 60  0001 C CNN "Package"
+F 7 "Farnell" H 5300 2300 60  0001 C CNN "Supplier"
+F 8 "2447598" H 5300 2300 60  0001 C CNN "Order Code"
+F 9 "Mouser" H 5300 2300 60  0001 C CNN "Alt. Supplier"
+F 10 "667-ERJ-6GEYJ1R0V" H 5300 2300 60  0001 C CNN "Alt. Order Code"
+F 11 "1Ω/1% 0805 resistor" H 5300 2300 60  0001 C CNN "Note"
 	1    5300 2300
 	1    0    0    -1
@@
 F 2 "Resistors_SMD:R_0805" V 5230 4400 50  0001 C CNN
 F 3 "" H 5300 4400 50  0000 C CNN
+F 4 "MCWR08W1R00FTL" H 5300 4400 60  0001 C CNN "Part Number"
+F 5 "Multicomp" H 5300 4400 60  0001 C CNN "Manufacturer"
+F 6 "0805" H 5300 4400 60  0001 C CNN "Package"
+F 7 "Farnell" H 5300 4400 60  0001 C CNN "Supplier"
+F 8 "2447598" H 5300 4400 60  0001 C CNN "Order Code"
+F 9 "Mouser" H 5300 4400 60  0001 C CNN "Alt. Supplier"
+F 10 "667-ERJ-6GEYJ1R0V" H 5300 4400 60  0001 C CNN "Alt. Order Code"
+F 11 "1Ω/1% 0805 resistor" H 5300 4400 60  0001 C CNN "Note"
 	1    5300 4400
 	1    0    0    -1

Commit message: Re-referenced components
Parts:
- C47, C48: value 1u/10V -> 1u/25V; Alt. Order Code 710-885012106010 -> 603-CC603KRX7R8BB105; Manufacturer Multicomp -> Murata; Note 1μF/10V X5R 0603 ceramic capacitor -> 1μF/25V X7R 0603 ceramic capacitor; Order Code 1759399 -> 2470425; Part Number MC0603X105K100CT -> GCM188R71E105KA64D
Changed lines of the file:
@@
-	1    0    0    -1
-$EndComp
-$Comp
-L C C47
-U 1 1 5573B996
-P 4900 2700
-F 0 "C47" H 4950 2800 50  0000 L CNN
-F 1 "1u/10V" H 4950 2600 50  0000 L CNN
-F 2 "Capacitors_SMD:C_0603" H 4938 2550 30  0001 C CNN
-F 3 "" H 4900 2700 60  0000 C CNN
-F 4 "MC0603X105K100CT" H 4900 2700 60  0001 C CNN "Part Number"
-F 5 "Multicomp" H 4900 2700 60  0001 C CNN "Manufacturer"
-F 6 "0603" H 4900 2700 60  0001 C CNN "Package"
-F 7 "Farnell" H 4900 2700 60  0001 C CNN "Supplier"
-F 8 "1759399" H 4900 2700 60  0001 C CNN "Order Code"
-F 9 "Mouser" H 4900 2700 60  0001 C CNN "Alt. Supplier"
-F 10 "710-885012106010" H 4900 2700 60  0001 C CNN "Alt. Order Code"
-F 11 "1μF/10V X5R 0603 ceramic capacitor" H 4900 2700 60  0001 C CNN "Note"
-	1    4900 2700
 	1    0    0    -1
 $EndComp
@@
 	2900 2000 2900 2600
 $Comp
-L GNDA #PWR48
+L GNDA #PWR048
 U 1 1 5573B9A8
 P 2900 3000
-F 0 "#PWR48" H 2900 2750 60  0001 C CNN
+F 0 "#PWR048" H 2900 2750 60  0001 C CNN
 F 1 "GNDA" H 2900 2850 60  0000 C CNN
 F 2 "" H 2900 3000 60  0000 C CNN
@@
 $EndComp
 $Comp
-L GNDA #PWR52
+L GNDA #PWR049
 U 1 1 5573B9AE
 P 4900 3000
-F 0 "#PWR52" H 4900 2750 60  0001 C CNN
+F 0 "#PWR049" H 4900 2750 60  0001 C CNN
 F 1 "GNDA" H 4900 2850 60  0000 C CNN
 F 2 "" H 4900 3000 60  0000 C CNN
@@
 	2900 3000 2900 2900
 $Comp
-L GNDA #PWR54
+L GNDA #PWR050
 U 1 1 5573B9C2
 P 5300 3000
-F 0 "#PWR54" H 5300 2750 60  0001 C CNN
+F 0 "#PWR050" H 5300 2750 60  0001 C CNN
 F 1 "GNDA" H 5300 2850 60  0000 C CNN
 F 2 "" H 5300 3000 60  0000 C CNN
@@
 	1    0    0    -1
 $EndComp
-$Comp
-L C C48
-U 1 1 5573BE4D
-P 4900 4800
-F 0 "C48" H 4950 4900 50  0000 L CNN
-F 1 "1u/10V" H 4950 4700 50  0000 L CNN
-F 2 "Capacitors_SMD:C_0603" H 4938 4650 30  0001 C CNN
-F 3 "" H 4900 4800 60  0000 C CNN
-F 4 "MC0603X105K100CT" H 4900 4800 60  0001 C CNN "Part Number"
-F 5 "Multicomp" H 4900 4800 60  0001 C CNN "Manufacturer"
-F 6 "0603" H 4900 4800 60  0001 C CNN "Package"
-F 7 "Farnell" H 4900 4800 60  0001 C CNN "Supplier"
-F 8 "1759399" H 4900 4800 60  0001 C CNN "Order Code"
-F 9 "Mouser" H 4900 4800 60  0001 C CNN "Alt. Supplier"
-F 10 "710-885012106010" H 4900 4800 60  0001 C CNN "Alt. Order Code"
-F 11 "1μF/10V X5R 0603 ceramic capacitor" H 4900 4800 60  0001 C CNN "Note"
-	1    4900 4800
-	1    0    0    -1
-$EndComp
 Wire Wire Line
 	2700 4100 3500 4100
@@
 	2900 4100 2900 4700
 $Comp
-L GNDA #PWR49
+L GNDA #PWR051
 U 1 1 5573BE5B
 P 2900 5100
-F 0 "#PWR49" H 2900 4850 60  0001 C CNN
+F 0 "#PWR051" H 2900 4850 60  0001 C CNN
 F 1 "GNDA" H 2900 4950 60  0000 C CNN
 F 2 "" H 2900 5100 60  0000 C CNN
@@
 $EndComp
 $Comp
-L GNDA #PWR53
+L GNDA #PWR052
 U 1 1 5573BE61
 P 4900 5100
-F 0 "#PWR53" H 4900 4850 60  0001 C CNN
+F 0 "#PWR052" H 4900 4850 60  0001 C CNN
 F 1 "GNDA" H 4900 4950 60  0000 C CNN
 F 2 "" H 4900 5100 60  0000 C CNN
@@
 	2900 5100 2900 5000
 $Comp
-L GNDA #PWR55
+L GNDA #PWR053
 U 1 1 5573BE72
 P 5300 5100
-F 0 "#PWR55" H 5300 4850 60  0001 C CNN
+F 0 "#PWR053" H 5300 4850 60  0001 C CNN
 F 1 "GNDA" H 5300 4950 60  0000 C CNN
 F 2 "" H 5300 5100 60  0000 C CNN
@@
 	3400 2600 3400 3400
 $Comp
-L GNDA #PWR50
+L GNDA #PWR054
 U 1 1 5573C48B
 P 3400 3400
-F 0 "#PWR50" H 3400 3150 60  0001 C CNN
+F 0 "#PWR054" H 3400 3150 60  0001 C CNN
 F 1 "GNDA" H 3400 3250 60  0000 C CNN
 F 2 "" H 3400 3400 60  0000 C CNN
@@
 	3400 4700 3400 5500
 $Comp
-L GNDA #PWR51
+L GNDA #PWR055
 U 1 1 5573C579
 P 3400 5500
-F 0 "#PWR51" H 3400 5250 60  0001 C CNN
+F 0 "#PWR055" H 3400 5250 60  0001 C CNN
 F 1 "GNDA" H 3400 5350 60  0000 C CNN
 F 2 "" H 3400 5500 60  0000 C CNN
@@
 Text Notes 5650 2350 0    60   ~ 0
 1Ω ESR resistor for output stability
+$Comp
+L C C47
+U 1 1 56F2D0D4
+P 4900 2700
+F 0 "C47" H 4950 2800 50  0000 L CNN
+F 1 "1u/25V" H 4950 2600 50  0000 L CNN
+F 2 "Capacitors_SMD:C_0603" H 4938 2550 30  0001 C CNN
+F 3 "" H 4900 2700 60  0000 C CNN
+F 4 "GCM188R71E105KA64D" H 4900 2700 60  0001 C CNN "Part Number"
+F 5 "Murata" H 4900 2700 60  0001 C CNN "Manufacturer"
+F 6 "0603" H 4900 2700 60  0001 C CNN "Package"
+F 7 "Farnell" H 4900 2700 60  0001 C CNN "Supplier"
+F 8 "2470425" H 4900 2700 60  0001 C CNN "Order Code"
+F 9 "Mouser" H 4900 2700 60  0001 C CNN "Alt. Supplier"
+F 10 "603-CC603KRX7R8BB105" H 4900 2700 60  0001 C CNN "Alt. Order Code"
+F 11 "1μF/25V X7R 0603 ceramic capacitor" H 4900 2700 60  0001 C CNN "Note"
+	1    4900 2700
+	1    0    0    -1
+$EndComp
+$Comp
+L C C48
+U 1 1 56F2D0F5
+P 4900 4800
+F 0 "C48" H 4950 4900 50  0000 L CNN
+F 1 "1u/25V" H 4950 4700 50  0000 L CNN
+F 2 "Capacitors_SMD:C_0603" H 4938 4650 30  0001 C CNN
+F 3 "" H 4900 4800 60  0000 C CNN
+F 4 "GCM188R71E105KA64D" H 4900 4800 60  0001 C CNN "Part Number"
+F 5 "Murata" H 4900 4800 60  0001 C CNN "Manufacturer"
+F 6 "0603" H 4900 4800 60  0001 C CNN "Package"
+F 7 "Farnell" H 4900 4800 60  0001 C CNN "Supplier"
+F 8 "2470425" H 4900 4800 60  0001 C CNN "Order Code"
+F 9 "Mouser" H 4900 4800 60  0001 C CNN "Alt. Supplier"
+F 10 "603-CC603KRX7R8BB105" H 4900 4800 60  0001 C CNN "Alt. Order Code"
+F 11 "1μF/25V X7R 0603 ceramic capacitor" H 4900 4800 60  0001 C CNN "Note"
+	1    4900 4800
+	1    0    0    -1
+$EndComp
 $EndSCHEMATC
